Commit message: working sonar in uuv simulator

File: uuv_descriptions/robots/rexrov_test.xacro (robot description, xacro)
@@ -20,4 +20,5 @@
   <xacro:include filename="$(find uuv_descriptions)/urdf/rexrov.gazebo.xacro"/>
   <xacro:forward_looking_sonar
+      topic="lol"
       namespace="${namespace}"
       suffix="horiz"
@@ -31,17 +32,4 @@
     <inertia ixx="0.00001" ixy="0.0" ixz="0.0" iyy="0.00001" iyz="0.0" izz="0.00001" />
     <origin xyz="1.15 0 0.35" rpy="0 0 0"/>
-  </xacro:forward_looking_sonar>
-  <xacro:forward_looking_sonar
-      namespace="${namespace}"
-      suffix="vert"
-      parent_link="${namespace}/base_link"
-      mass="0.015"
-      update_rate="40"
-      samples="512"
-      fov="2.26893"
-      width="768"
-      height="768">
-    <inertia ixx="0.00001" ixy="0.0" ixz="0.0" iyy="0.00001" iyz="0.0" izz="0.00001" />
-    <origin xyz="1.15 0 0.45" rpy="1.5707 0 0"/>
   </xacro:forward_looking_sonar>
   <!-- Create the RexROV vehicle -->

File: uuv_sensor_plugins/uuv_sensor_ros_plugins/urdf/sonar_snippets.xacro (robot description, xacro)
@@ -194,5 +194,7 @@
         </camera>
 	    <plugin filename="libimage_sonar_ros_plugin.so" name="forward_sonar${suffix}_controller">
-		  <topicName>${topic}</topicName>
+		  <!--topicName>${topic}</topicName-->
+                <sonarGroupTopicName>forward_sonar_${suffix}</sonarGroupTopicName>
+          <imageTopicName>forward_sonar_${suffix}/raw_image</imageTopicName>
           <frameName>forward_sonar${suffix}_optical_frame</frameName>
         </plugin>

Commit message: Adding second sonar to ROV

File: uuv_descriptions/robots/rexrov_test.xacro (robot description, xacro)
@@ -21,5 +21,5 @@
   <xacro:forward_looking_sonar
       topic="lol"
-      namespace="${namespace}"
+      namespace="${namespace}/horizontal_sonar"
       suffix="horiz"
       parent_link="${namespace}/base_link"
@@ -31,5 +31,19 @@
       height="768">
     <inertia ixx="0.00001" ixy="0.0" ixz="0.0" iyy="0.00001" iyz="0.0" izz="0.00001" />
-    <origin xyz="1.15 0 0.35" rpy="0 0 0"/>
+    <origin xyz="1.15 0 0.25" rpy="0 0 0"/>
+  </xacro:forward_looking_sonar>
+  <xacro:forward_looking_sonar
+      topic="lol"
+      namespace="${namespace}/vertical_sonar"
+      suffix="vert"
+      parent_link="${namespace}/base_link"
+      mass="0.015"
+      update_rate="40"
+      samples="512"
+      fov="2.26893"
+      width="768"
+      height="768">
+    <inertia ixx="0.00001" ixy="0.0" ixz="0.0" iyy="0.00001" iyz="0.0" izz="0.00001" />
+    <origin xyz="1.15 0 0.35" rpy="1.5708 0 0"/>
   </xacro:forward_looking_sonar>
   <!-- Create the RexROV vehicle -->
