Commit message: Moving IMU to align with sonar frame

File: uuv_descriptions/urdf/rexrov_sensors.xacro (robot description, xacro)
@@ -35,5 +35,5 @@
     parent_link="${namespace}/base_link"
     inertial_reference_frame="${inertial_reference_frame}">
-    <origin xyz="0 0 0" rpy="0 0 0"/>
+    <origin xyz="1.15 0 0" rpy="0 0 0"/>
   </xacro:default_imu_macro>
   <!-- Mount a camera -->

Commit message: Changed DVL location to center

File: uuv_descriptions/urdf/rexrov_sensors.xacro (robot description, xacro)
@@ -18,5 +18,5 @@
     parent_link="${namespace}/base_link"
     inertial_reference_frame="${inertial_reference_frame}">
-    <origin xyz="-1.4 0 -0.312" rpy="0 ${0.5*pi} 0"/>
+    <origin xyz="0 0 0" rpy="0 ${0.5*pi} 0"/>
   </xacro:default_dvl_macro>
   <!-- Magnetometer  -->

Commit message: Updating DVL location, following Ivana's updates

File: uuv_descriptions/urdf/rexrov_sensors.xacro (robot description, xacro)
@@ -18,5 +18,5 @@
     parent_link="${namespace}/base_link"
     inertial_reference_frame="${inertial_reference_frame}">
-    <origin xyz="-1.4 0 -0.312" rpy="0 ${0.5*pi} 0"/>
+    <origin xyz="0 0 0" rpy="0 ${0.5*pi} 0"/>
   </xacro:default_dvl_macro>
   <!-- Magnetometer  -->
@@ -35,5 +35,5 @@
     parent_link="${namespace}/base_link"
     inertial_reference_frame="${inertial_reference_frame}">
-    <origin xyz="1.15 0 0" rpy="0 0 0"/>
+    <origin xyz="0 0 0" rpy="0 0 0"/>
   </xacro:default_imu_macro>
   <!-- Mount a camera -->

Commit message: costum camera and somar placement

File: uuv_descriptions/urdf/rexrov_sensors.xacro (robot description, xacro)
@@ -39,5 +39,5 @@
   <!-- Mount a camera -->
   <xacro:default_camera namespace="${namespace}" parent_link="${namespace}/base_link" suffix="">
-    <origin xyz="1.15 0 0.4" rpy="0 0.6 0"/>
+    <origin xyz="0.55 0 0.17" rpy="1.5707 0.0 0"/>
   </xacro:default_camera>
   <xacro:default_camera namespace="${namespace}" parent_link="${namespace}/base_link" suffix="right">

File: uuv_sensor_plugins/uuv_sensor_ros_plugins/urdf/sonar_snippets.xacro (robot description, xacro)
@@ -162,9 +162,9 @@
         <origin xyz="0 0 0" rpy="0 0 0" />
       </inertial>
-      <visual>
+      <!--visual>
         <geometry>
           <mesh filename="file://$(find uuv_sensor_ros_plugins)/meshes/oe14-372.dae" scale="1 1 1"/>
         </geometry>
-      </visual>
+      </visual-->
       <xacro:no_collision/>
     </link>
